Commit message: Remove the vendor identifier from the shipped task and re-validate
The robot's calibration file carried a vendor-specific name, in its filename, in
its robot element, in five sensor-mount joint names and in a control block, and
that file ships inside the agent container. Renamed to robot_frames.urdf with
the robot as survey_robot and the joints as lidar_hesai_to_base_link,
livox_{front,rear,left,right}_to_base_link. Every reference updated: the
instruction, the environment Dockerfile, the data README, solve.sh, the launch
file, the data tooling and the design docs.

Re-validated rather than assumed, because the rename touches files the agent
reads and the solution depends on: 22/22 static checks and oracle reward 1 on
the GCP VM with the environment image rebuilt (re-accumulation 0.812/0.996,
model 0.813/0.992). Evidence in docs/runs/rename-oracle/.

The 2.9 GB recording was scanned in full for the identifier and its variants:
zero matches, so no frame name, schema or metadata record in the published
dataset carries it, and the dataset needs no change.

Agent transcripts under docs/runs/ still contain the old name because the agents
read and quoted that file during their trials. They are evidence of what
happened and are deliberately left unedited.

Co-Authored-By: Claude Opus 5 <noreply@anthropic.com>

File: tasks/aircraft-orbit-mapping/environment/data/robot_frames.urdf (robot description, URDF)
Before this commit: robot i-trek, 24 links, 23 joints
Joints:
- removed joint itrek_lidar_hesai_to_base_link
- removed joint itrek_livox_front_to_base_link
- removed joint itrek_livox_left_to_base_link
- removed joint itrek_livox_rear_to_base_link
- removed joint itrek_livox_right_to_base_link
- added joint lidar_hesai_to_base_link: type fixed, parent base_link, child hesai, origin xyz=0 0 0.543963814026 rpy=0 0 1.5708
- added joint livox_front_to_base_link: type fixed, parent base_link, child livox_front, origin xyz=0.428807815738 0 0.365184072526 rpy=-0.872665 0 -1.5708
- added joint livox_left_to_base_link: type fixed, parent base_link, child livox_left, origin xyz=0 0.349484353354 0.355127188398 rpy=-0.872665 0 0
- added joint livox_rear_to_base_link: type fixed, parent base_link, child livox_rear, origin xyz=-0.428807815738 0 0.365184072526 rpy=-0.872665 0 1.5708
- added joint livox_right_to_base_link: type fixed, parent base_link, child livox_right, origin xyz=0 -0.349484353354 0.355127188398 rpy=0.872665 0 0
